File: Eros Tracker BNO086 IMU.kicad_sch (KiCad schematic)
At the start: 7 parts, among them U4 BNO086

Commit message: Rev E release
Connections:
- net +3V3: now also RN1.5, RN1.6; no longer RN1.7, RN1.7
- net at U4.15 (ENV_SCL): now also RN1.4; no longer RN1.2
- net at U4.16 (ENV_SDA): now also RN1.3; no longer RN1.2
