File: Eros Tracker Connectors.kicad_sch (KiCad schematic)
At the start: 14 parts, among them J1 USB4110-GF-A, J3 B2B-PH-SM4-TB(LF)(SN), J4 24881, J5 24881, J6 24881, J7 24881

Commit message: Rev D realease
Parts:
- J10, J9: symbol Eros Tracker:Power_Pad -> Eros Tracker:Power_Pad_0.8mm; Manufacturer_Name (none) -> Total Element
- J11, J8: symbol Eros Tracker:Power_Pad -> Eros Tracker:Power_Pad_1.0mm; Manufacturer_Name (none) -> Total Element
Changed lines of the file:
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@@
     )
   )
-  (symbol (lib_id "Eros Tracker:Power_Pad") (at 223.52 116.84 0) (unit 1)
+  (symbol (lib_id "Eros Tracker:Power_Pad_1.0mm") (at 223.52 116.84 0) (unit 1)
     (in_bom yes) (on_board yes) (dnp no) (fields_autoplaced)
     (property "Reference" "J8" (at 226.06 117.475 0)
@@
     )
     (property "Datasheet" "https://totalelement.com/collections/steel-discs/products/3-8-inch-steel-disc-blank-metal-strike-plates-250-pack" (at 223.52 116.84 0)
+      (effects (font (size 1.27 1.27)) hide)
+    )
+    (property "Manufacturer_Name" "Total Element" (at 223.52 116.84 0)
       (effects (font (size 1.27 1.27)) hide)
     )
@@
     )
   )
-  (symbol (lib_id "Eros Tracker:Power_Pad") (at 223.52 125.73 0) (unit 1)
+  (symbol (lib_id "Eros Tracker:Power_Pad_0.8mm") (at 223.52 125.73 0) (unit 1)
     (in_bom yes) (on_board yes) (dnp no) (fields_autoplaced)
     (property "Reference" "J9" (at 226.06 126.365 0)
@@
       (effects (font (size 1.27 1.27)) hide)
     )
+    (property "Manufacturer_Name" "Total Element" (at 223.52 125.73 0)
+      (effects (font (size 1.27 1.27)) hide)
+    )
     (pin "1")
     (instances
@@
     )
   )
-  (symbol (lib_id "Eros Tracker:Power_Pad") (at 242.57 116.84 0) (unit 1)
+  (symbol (lib_id "Eros Tracker:Power_Pad_0.8mm") (at 242.57 116.84 0) (unit 1)
     (in_bom yes) (on_board yes) (dnp no) (fields_autoplaced)
     (property "Reference" "J10" (at 245.11 117.475 0)
@@
     )
     (property "Datasheet" "https://totalelement.com/collections/steel-discs/products/3-8-inch-steel-disc-blank-metal-strike-plates-250-pack" (at 242.57 116.84 0)
+      (effects (font (size 1.27 1.27)) hide)
+    )
+    (property "Manufacturer_Name" "Total Element" (at 242.57 116.84 0)
       (effects (font (size 1.27 1.27)) hide)
     )
@@
     )
   )
-  (symbol (lib_id "Eros Tracker:Power_Pad") (at 242.57 125.73 0) (unit 1)
+  (symbol (lib_id "Eros Tracker:Power_Pad_1.0mm") (at 242.57 125.73 0) (unit 1)
     (in_bom yes) (on_board yes) (dnp no) (fields_autoplaced)
     (property "Reference" "J11" (at 245.11 126.365 0)
@@
       (effects (font (size 1.27 1.27)) hide)
     )
+    (property "Manufacturer_Name" "Total Element" (at 242.57 125.73 0)
+      (effects (font (size 1.27 1.27)) hide)
+    )

Commit message: Rev E release
Parts:
- removed R13 (x2): 5k1, Resistor_SMD:R_0402_1005Metric, symbol Device:R_US
- added D5: PESD15VL2BT,215, Eros Tracker:SOT95P230X110-3N, symbol Eros Tracker:PESD15VL2BT,215
- D3: value PESD5V2S2UT,215 -> PESD15VL2BT,215; symbol Eros Tracker:PESD5V2S2UT,215 -> Eros Tracker:PESD15VL2BT,215; Manufacturer_Part_Number PESD5V2S2UT,215 -> PESD15VL2BT,215; Mouser Part Number 771-PESD5V2S2UT-T/R -> 771-PESD15VL2BT-T/R; Mouser Price/Stock https://www.mouser.co.uk/ProductDetail/Nexperia/PESD5V2S2UT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 -> https://www.mouser.com/ProductDetail/Nexperia/PESD15VL2BT21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
- J10, J9: value ~ -> 0.8mm
- J11, J8: value ~ -> 1mm
Connections:
- net GND: now also D5.3
- net VBUS_OUT: now also D5.1; no longer FL1.11, FL1.4 (ID)
- net USB_CC1: now reaches J1.A5 (CC1)
- net USB_CC2: now reaches J1.B5 (CC2)
- new net: FL1.11, FL1.4 (ID)
- no-connect marks 4 -> 5
Other:
- moved on the sheet: J4, J5, J6, J7
