File: Eros Tracker Microcontroller.kicad_sch (KiCad schematic)
At the start: 24 parts, among them M1 LCM04084521-B1, Q1 NX138BKSX, Q2 NX138BKSX, Q3 DMP31D7LDW-7, SW1 EVQ-P7A01P, U1 ESP32-C3-MINI-1-N4

Commit message: Rev D realease
Parts:
- removed D1: BAT54C, Package_TO_SOT_SMD:SOT-23, symbol Diode:BAT54C
- added D1: BAS40VYX, Eros Tracker:SOT65P210X110-6N, symbol Eros Tracker:BAS40VYX
- added R10, R15: 10k 1%, Resistor_SMD:R_0402_1005Metric, symbol Device:R_US
- JP1: Manufacturer_Name (none) -> Total Element
- M1: now not fitted; now left out of the parts list
- U1: footprint Eros Tracker:XCVR_ESP32-C3-MINI-1-N4 -> XCVR_ESP32-C3-MINI-1-N4; Height (none) -> 2.55; MANUFACTURER Espressif Systems -> (none); MAXIMUM_PACKAGE_HEIGHT 2.55mm -> (none); PARTREV v1.0 -> (none); STANDARD Manufacturer Recommendations -> (none)
Connections:
- net +3V3: now also R10.1
- net +BATT: now also D1.4 (K3)
- net GND: now also R15.2
- net TACT_MOTOR: now also R15.1
- net ~{BAT_STAT_CHARGING}: now also D1.6 (K1), R10.2; no longer Q2.6 (D1), Q3.2 (G1), R9.2
- net at M1.2 (-), Q1.3 (D2): now also D1.3 (A3)
- net ~{BUTTON_INPUT} renamed BUTTON_INPUT
- new net: D1.1 (A1), Q2.6 (D1), Q3.2 (G1), R9.2
- no-connect marks 0 -> 2
Other:
- moved on the sheet: C4, LED1, LED2, Q3B, R11, R15

Commit message: Rev E release
Parts:
- added C11: 0.1uF, Capacitor_SMD:C_0402_1005Metric, symbol Device:C
- added R21: 10k 1%, Resistor_SMD:R_0402_1005Metric, symbol Device:R_US
- added TP5: TestPoint, TestPoint:TestPoint_Pad_D1.0mm, symbol Connector:TestPoint
- added U6: FUSB302BUCX, Eros Tracker:BGA9C40P3X3_122X126X53, symbol Eros Tracker:FUSB302BUCX
- U1: footprint XCVR_ESP32-C3-MINI-1-N4 -> Eros Tracker:XCVR_ESP32-C3-MINI-1-N4
- renumbered C4 to C1, R11 to R1, R11 to R2, R15 to R24, R9 to R3, R13 to R4, R15 to R5, R13 to R6, R15 to R7, R15 to R8, R15 to R9, TP2 to TP10, TP2 to TP12, TP2 to TP9
Connections:
- net +3V3: now also R21.1
- net GND: now also C11.2, U6.C2 (GND)
- net I2C_SCL: now also U6.B3 (SCL)
- net I2C_SDA: now also U6.C3 (SDA)
- net IMU_RESET renamed BAT_CHRG_DONE
- net ~{BAT_STAT_CHARGING} renamed ~{POWER GOOD}
- net ~{POWER GOOD}: no longer U1.18 (IO4,ADC1_CH4,FSPIHD,MTMS)
- net ~{BAT_STAT_CHRG_DONE} renamed CHRG_INT
- new net: TP5.1, U6.B1 (VCONN)
- new net +4V5: C11.1, U6.A3 (VDD)
- new net USB_CC1: U6.C1 (CC1)
- new net USB_CC2: U6.A1 (CC2)
- new net USB_PD_INT: R21.2, U1.18 (IO4,ADC1_CH4,FSPIHD,MTMS), U6.B2 (INT_N)
- new net VBUS: U6.A2 (VBUS)
Other:
- moved on the sheet: LED1, LED2, Q3B, R24, R8, R9
