File: Eros Tracker Power - Battery.kicad_sch (KiCad schematic)
At the start: 23 parts, among them Q4 DMP2240UDM-7, Q5 DMC1028UVT-7, Q6 DMC1028UVT-7, Q7 NX138BKSX, U2 TPS62A01A, U3 MCP73834-FCI/MF

Commit message: Rev D realease
Parts:
- added C10: DNI, Capacitor_SMD:C_0805_2012Metric, symbol Device:C
- added C7, C9: 22uF, Capacitor_SMD:C_0805_2012Metric, symbol Device:C
- added C8: DNI, Capacitor_SMD:C_0603_1608Metric, symbol Device:C
- added L2: 2.2uH, Eros Tracker:DFE2HCAH1R0MJ0L, symbol Device:L
- added R10, R25: 10k 1%, Resistor_SMD:R_0402_1005Metric, symbol Device:R_US
- added R21: 100k, Resistor_SMD:R_0402_1005Metric, symbol Device:R_US
- added U5: TLV61070ADBVR, Eros Tracker:SOT95P280X145-6N, symbol Eros Tracker:TLV61070ADBVR
- C3: Manufacturer_Part_Number GRM21BZ70J226ME44L -> GRM21BZ71A226ME15L; Mouser Part Number 81-GRM21BZ70J226ME4L -> 81-GRM21BZ71A226ME5L; Mouser Price/Stock https://www.mouser.com/ProductDetail/Murata-Electronics/GRM21BZ70J226ME44L?qs=gt1LBUVyoHk1niSPiXLfGQ%3D%3D -> https://www.mouser.com/ProductDetail/Murata-Electronics/GRM21BZ71A226ME15L?qs=Ey7%2FXF42M3ejDq7iqlmWWw%3D%3D
- R11: value 10k 1% -> 100k; Manufacturer_Part_Number RT0402FRE0710KL -> RT0402FRE07100KL; Mouser Part Number 603-RT0402FRE0710KL -> 603-RT0402FRE07100KL; Mouser Price/Stock https://www.mouser.com/ProductDetail/YAGEO/RT0402FRE0710KL?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 -> https://www.mouser.com/ProductDetail/YAGEO/RT0402FRE07100KL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
Connections:
- net +3V3: now also R10.1; no longer Q7.2 (G1)
- net GND: now also Q7.1 (S1), C10.2, C7.2, C9.2, R25.2, U5.2 (GND)
- net VBUS: now also C7.1, L2.1, U5.6 (VIN); no longer Q4.2 (S2)
- net VBUS_OUT: now also C10.1, C8.1, C9.1, R21.1, U5.5 (VOUT); no longer Q4.4 (D2)
- net ~{BAT_STAT_CHRG_DONE}: now also Q7.2 (G1), R10.2; no longer Q7.1 (S1)
- net at Q7.6 (D1), R11.2: now also U5.3 (EN); no longer Q4.3 (G2)
- new net: L2.2, U5.1 (SW)
- new net: C8.2, R21.2, R25.1, U5.4 (FB)
- no-connect marks 1 -> 4
Other:
- note removed: "Pulled up by MCU pin"
- moved on the sheet: D2, Q4A, Q4B, Q5A, Q5B, Q6A, Q6B, Q7A, R12, R15, R16, TP3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

Commit message: Rev E release
Parts:
- removed Q7: NX138BKSX, Eros Tracker:SOT65P210X110-6N, symbol Eros Tracker:NX138BKSX
- removed R10, R12: 10k 1%, Resistor_SMD:R_0402_1005Metric, symbol Device:R_US
- removed R11, R21: 100k, Resistor_SMD:R_0402_1005Metric, symbol Device:R_US
- removed U3: MCP73834-FCI/MF, Eros Tracker:MCP73834-FCI-MF, symbol Eros Tracker:MCP73834-FCI/MF
- removed U5: TLV61070ADBVR, Eros Tracker:SOT95P280X145-6N, symbol Eros Tracker:TLV61070ADBVR
- added C12: 4.7uF, Capacitor_SMD:C_0603_1608Metric, symbol Device:C
- added Q1: NX138BKSX, Eros Tracker:SOT65P210X110-6N, symbol Eros Tracker:NX138BKSX
- added R20: 10k 1%, Resistor_SMD:R_0402_1005Metric, symbol Device:R_US
- added TH1: 10k, Resistor_SMD:R_0402_1005Metric, symbol Device:Thermistor_NTC_US
- added TP6, TP7: TestPoint, TestPoint:TestPoint_Pad_D1.0mm, symbol Connector:TestPoint
- added U3: BQ24196RGER, Eros Tracker:QFN50P400X400X100-25N-D, symbol Eros Tracker:BQ24196RGER
- C10: value DNI -> 22uF; Manufacturer_Name (none) -> Murata; Manufacturer_Part_Number (none) -> GRM21BZ71A226ME15L; Mouser Part Number (none) -> 81-GRM21BZ71A226ME5L; Mouser Price/Stock (none) -> https://www.mouser.com/ProductDetail/Murata-Electronics/GRM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; now fitted; now in the parts list
- C2: footprint Capacitor_SMD:C_0805_2012Metric -> Capacitor_SMD:C_0603_1608Metric; Manufacturer_Part_Number GRM21BR71C475KE51L -> GRM188Z71C475KE21D; Mouser Part Number 81-GRM21BR71C475KE1L -> 81-GRM188Z71C475KE1D; Mouser Price/Stock https://www.mouser.com/ProductDetail/Murata-Electronics/GRM21BR71C475KE51L?qs=eeBpzGFlv%252B%252BCR4pji%2FtFiA%3D%3D -> https://www.mouser.com/ProductDetail/Murata-Electronics/GRM188Z71C475KE21D?qs=d0WKAl%252BL4KajNOvalhHKtQ%3D%3D
- C7: value 22uF -> 1uF; footprint Capacitor_SMD:C_0805_2012Metric -> Capacitor_SMD:C_0603_1608Metric; Manufacturer_Name Murata -> TAIYO YUDEN; Manufacturer_Part_Number GRM21BZ71A226ME15L -> MLASU168AB7105KTNA01; Mouser Part Number 81-GRM21BZ71A226ME5L -> 963-MLASU168AB7105KT; Mouser Price/Stock https://www.mouser.com/ProductDetail/Murata-Electronics/GRM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 -> https://www.mouser.com/ProductDetail/TAIYO-YUDEN/MLASU168AB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
- C8: value DNI -> 0.47uF; footprint Capacitor_SMD:C_0603_1608Metric -> Capacitor_SMD:C_0402_1005Metric; Manufacturer_Name (none) -> YAGEO; Manufacturer_Part_Number (none) -> CC0402KRX7R6BB474; Mouser Part Number (none) -> 603-CC0402KR6BB474; Mouser Price/Stock (none) -> https://www.mouser.com/ProductDetail/YAGEO/CC0402KRX7R6BB47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; now fitted; now in the parts list
- C9: value 22uF -> 6.8uF; footprint Capacitor_SMD:C_0805_2012Metric -> Capacitor_SMD:C_1210_3225Metric; Manufacturer_Part_Number GRM21BZ71A226ME15L -> C3225X7R1E685K250AB; Mouser Part Number 81-GRM21BZ71A226ME5L -> 810-C3225X7R1E685K11; Mouser Price/Stock https://www.mouser.com/ProductDetail/Murata-Electronics/GRM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 -> https://www.mouser.com/ProductDetail/TDK/C3225X7R1E685K250A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
- L2: footprint Eros Tracker:DFE2HCAH1R0MJ0L -> Eros Tracker:1277ASH100MP2; Manufacturer_Part_Number DFE252012F-2R2M=P2 -> DFE322512F-2R2M=P2; Mouser Part Number 81-DFE252012F-2R2MP2 -> 81-DFE322512F-2R2MP2; Mouser Price/Stock https://www.mouser.com/ProductDetail/Murata-Electronics/DFE252012F-2R2M%3dP2?qs=ty6qhqyUUEuYhdA0a9%2F0aw%3D%3D -> https://www.mouser.com/ProductDetail/Murata-Electronics/DFE322512F-2R2M%3dP2?qs=AQlKX63v8RugBXCoLvLHRA%3D%3D
- R17: value 835R -> 6K65; footprint Resistor_SMD:R_0805_2012Metric -> Resistor_SMD:R_0402_1005Metric; Manufacturer_Part_Number RT0805BRD07835RL -> RT0402DRE076K65L; Mouser Part Number 603-RT0805BRD07835RL -> 603-RT0402DRE076K65L; Mouser Price/Stock https://www.mouser.com/ProductDetail/YAGEO/RT0805BRD07835RL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 -> https://www.mouser.com/ProductDetail/YAGEO/RT0402DRE076K65L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
- renumbered R25 to R11
Connections:
- net +3V3: now also R20.1
- net +BATT: now also U3.13 (BAT), U3.14 (BAT_2); no longer Q4.5 (S1)
- net GND: now also R15.1, C12.2, Q1.1 (S1), TH1.2, U3.10 (ILIM), U3.17 (PGND), U3.18 (PGND_2), U3.2 (PSEL), U3.25 (EP), U3.8 (OTG), U3.9 (~{CE}); no longer R11.2, R16.2, R17.2
- net VBUS: now also Q4.5 (S1), R11.1, R16.2, U3.1 (VBUS), U3.24 (VBUS_2); no longer D2.2 (A), L2.1, Q4.1 (G1), R15.1
- net VBUS_OUT: now also D2.1 (K); no longer C10.1, C8.1, C9.1
- net at R17.1: now also C12.1, U3.22 (REGN)
- net at R18.1: now also R17.2, TH1.1, U3.11 (TS1), U3.12 (TS2)
- net +4V5: now reaches L2.2
- net +4V5: now also C10.1, C2.1, TP1.1, U2.3 (VIN), U2.4 (EN), U3.15 (SYS), U3.16 (SYS_2)
- net at C8.2: now also L2.1, U3.19 (SW), U3.20 (SW_2); no longer R11.1
- removed net VIN: C2.1, D2.1 (K), Q4.6 (D1), TP1.1, U2.3 (VIN), U2.4 (EN)
- net ~{BAT_STAT_CHRG_DONE} renamed BAT_CHRG_DONE
- net BAT_CHRG_DONE: now also Q1.2 (G1)
- new net: C9.1, U3.23 (PMID)
- new net: C8.1, U3.21 (BTST)
- new net: Q1.6 (D1), Q4.1 (G1), R11.2
- new net: D2.2 (A), Q4.6 (D1)
- new net CHRG_INT: R20.2, U3.7 (INT)
- new net I2C_SCL: TP6.1, U3.5 (SCL)
- new net I2C_SDA: TP7.1, U3.6 (SDA)
- new net ~{POWER GOOD}: U3.3 (~{PG})
- no-connect marks 4 -> 5
Other:
- note added: "4V5 - 18V5 Input"
- note added: "R13 = R14 * (Vout/0.6V - 1) = R13 * 4.5 for Vout = 3V3"
- note added: "R13, R14 0402, 1%"
- note removed: "DFE252012F-1R0M"
- note removed: "R5 = R6 * (Vout/0.6V - 1) = R6 * 4.5 for Vout = 3V3"
- note removed: "R5, R6 0805, 1%"
- moved on the sheet: C2, C3, C9, L1, Q4A, Q4B, Q5A, Q5B, Q6A, Q6B, R11, R13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
