File: Eros Tracker.kicad_pcb (KiCad board)
At the start: 4 copper layers, 50 x 50 mm, 69 parts, among them J1 USB4110-GF-A, J3 B2B-PH-SM4-TB(LF)(SN), J4 24881, J5 24881, J6 24881, J7 24881, M1 LCM04084521-B1, Q1 NX138BKSX, Q2 NX138BKSX, Q3 DMP31D7LDW-7, Q4 DMP2240UDM-7, Q5 DMC1028UVT-7, Q6 DMC1028UVT-7, SW1 EVQ-P7A01P, U1 ESP32-C3-MINI-1-N4, U2 TPS62A01A, U3 MCP73834-FCI/MF, U4 BNO086

Commit message: Rev D realease
Parts:
- added C10: DNI, Capacitor_SMD:C_0805_2012Metric, F.Cu at (171.8, 114.3)
- added C7: 22uF, Capacitor_SMD:C_0805_2012Metric, F.Cu at (164.0, 112.3)
- added C8: DNI, Capacitor_SMD:C_0603_1608Metric, F.Cu at (171.4, 111.0)
- added C9: 22uF, Capacitor_SMD:C_0805_2012Metric, F.Cu at (169.8, 114.3)
- added G2: ~, Eros Tracker:SomaticBananaLogo, F.Cu at (175.5, 84.3)
- added G3: ~, Eros Tracker:CE-Logo_7.0x5.0mm_SilkScreen, F.Cu at (175.5, 121.3)
- added L2: 2.2uH, Eros Tracker:DFE2HCAH1R0MJ0L, F.Cu at (161.6, 113.3)
- added R10: 10k 1%, Resistor_SMD:R_0402_1005Metric, F.Cu at (156.4, 101.3)
- added R20: 10k 1%, Resistor_SMD:R_0402_1005Metric, F.Cu at (156.4, 103.2)
- added R21: 10k 1%, Resistor_SMD:R_0402_1005Metric, F.Cu at (170.1, 111.1)
- added R25: 100k, Resistor_SMD:R_0402_1005Metric, F.Cu at (167.2, 110.4)
- added R7: 10k 1%, Resistor_SMD:R_0402_1005Metric, F.Cu at (179.8, 99.9)
- added U5: TLV61070ADBVR, Eros Tracker:SOT95P280X145-6N, F.Cu at (166.8, 113.3)
- D1: value BAT54C -> BAS40VYX; footprint Package_TO_SOT_SMD:SOT-23 -> Eros Tracker:SOT65P210X110-6N
- G1: renamed from LOGO; value LOGO -> ~
- G4: renamed from REF**; value FCC-Logo_7.3x6mm_SilkScreen -> ~; footprint Symbol:FCC-Logo_7.3x6mm_SilkScreen -> Eros Tracker:FCC-Logo_6.2x5.0mm_SilkScreen
- G5: renamed from REF**; value WEEE-Logo_4.2x6mm_SilkScreen -> ~
- G6: renamed from REF**; value OSHW-Logo2_7.3x6mm_SilkScreen -> ~
- R11: value 10k 1% -> 100k
- moved G6 12.9 mm to (153.4, 106.4)
- moved TP4 9.29 mm to (159.8, 118.0)
- moved FL1 1.20 mm to (165.5, 119.2)
- moved R12 1.06 mm to (151.7, 114.9), turned to 90 degrees
- moved R11 1.05 mm to (152.7, 114.9), turned to 90 degrees
- moved R23 0.56 mm to (167.3, 120.7), turned to 0 degrees
- moved D1 0.50 mm to (182.1, 96.6)
- moved Q1 0.50 mm to (182.0, 100.4)
- moved R22 0.46 mm to (163.3, 120.7), turned to 180 degrees
- moved G4 0.32 mm to (175.8, 126.7)
Connections:
- D1 pad 1: unconnected-(D1-Pad1) -> Net-(D1A-A1)
- D1 pad 2: Net-(M1--) -> unconnected-(D1B-A2-Pad2)
- D1 pad 3: +BATT -> Net-(D1C-A3)
- M1 pad 2: Net-(M1--) -> Net-(D1C-A3)
- Q1 pad 1: /Eros Tracker Microcontroller/~{BAT_STAT_CHRG_DONE} -> GND
- Q1 pad 2: +3V3 -> /Eros Tracker Microcontroller/~{BAT_STAT_CHRG_DONE}
- Q1 pad 3: Net-(M1--) -> Net-(D1C-A3)
- Q2 pad 6: /Eros Tracker Microcontroller/~{BAT_STAT_CHARGING} -> Net-(D1A-A1)
- Q3 pad 2: /Eros Tracker Microcontroller/~{BAT_STAT_CHARGING} -> Net-(D1A-A1)
- Q4 pad 2: /Eros Tracker Connectors/VBUS -> unconnected-(Q4B-S2-Pad2)
- Q4 pad 3: Net-(Q1A-D1) -> unconnected-(Q4B-G2-Pad3)
- Q4 pad 4: /Eros Tracker Connectors/VBUS_OUT -> unconnected-(Q4B-D2-Pad4)
- R3 pad 2: /Eros Tracker Microcontroller/~{BAT_STAT_CHARGING} -> Net-(D1A-A1)
Routing:
- net Net-(D1A-A1): track 0.00 -> 43.3 mm, vias 0 -> 2
- net Net-(M1--): track 9.75 -> 0.00 mm
- net /Eros Tracker Connectors/VBUS: track 71.0 -> 80.1 mm
- net Net-(D1C-A3): track 0.00 -> 8.95 mm
- net GND: track 51.1 -> 59.3 mm, vias 74 -> 77
- net /Eros Tracker Connectors/VBUS_OUT: track 24.7 -> 30.7 mm
- net Net-(U5-FB): track 0.00 -> 5.44 mm
- net Net-(Q1A-D1): track 35.7 -> 40.6 mm, vias 2 -> 3
- net /Eros Tracker Connectors/USB_D+: track 30.6 -> 35.2 mm
- net /Eros Tracker Connectors/USB_D-: track 29.9 -> 34.4 mm
- net /Eros Tracker Power & Battery/VIN: track 31.6 -> 34.7 mm
- net +3V3: track 29.6 -> 27.1 mm, vias 10 -> 11
- net Net-(FL1-D-_1): track 7.84 -> 5.78 mm
- net /Eros Tracker Connectors/POWER_VIN2: track 64.1 -> 62.1 mm
- net Net-(FL1-D+_1): track 7.09 -> 5.89 mm
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- added copper zone on F.Cu, net /Eros Tracker Connectors/VBUS
- added copper zone on F.Cu, net /Eros Tracker Connectors/VBUS_OUT
- added copper zone on F.Cu, net GND
- added copper zone on F.Cu, net Net-(U5-SW)
Other:
- board text added: "Banana Still Not To Scale"
- board text added: "Somatic Eros Rev. D"
- board text removed: "Somatic Eros Rev. C"

Commit message: Rev E release
Parts:
- removed R12: 10k 1%, Resistor_SMD:R_0402_1005Metric
- removed R22, R23: 5k1, Resistor_SMD:R_0402_1005Metric
- removed R25: 100k, Resistor_SMD:R_0402_1005Metric
- removed U5: TLV61070ADBVR, Eros Tracker:SOT95P280X145-6N
- added C11: 0.1uF, Capacitor_SMD:C_0402_1005Metric, F.Cu at (163.5, 112.1)
- added C12: 4.7uF, Capacitor_SMD:C_0603_1608Metric, F.Cu at (155.9, 105.2)
- added D5: PESD15VL2BT,215, Eros Tracker:SOT95P230X110-3N, F.Cu at (175.1, 123.3)
- added TH1: 10k, Resistor_SMD:R_0402_1005Metric, F.Cu at (151.5, 95.0)
- added TP5: TestPoint, TestPoint:TestPoint_Pad_D1.0mm, F.Cu at (165.4, 115.1)
- added TP6: TestPoint, TestPoint:TestPoint_Pad_D1.0mm, F.Cu at (171.9, 103.5)
- added TP7: TestPoint, TestPoint:TestPoint_Pad_D1.0mm, F.Cu at (171.9, 101.9)
- added U6: FUSB302BUCX, Eros Tracker:BGA9C40P3X3_122X126X53, F.Cu at (165.4, 112.4)
- C10: value DNI -> 22uF
- C2: footprint Capacitor_SMD:C_0805_2012Metric -> Capacitor_SMD:C_0603_1608Metric
- C7: value 22uF -> 1uF; footprint Capacitor_SMD:C_0805_2012Metric -> Capacitor_SMD:C_0603_1608Metric
- C8: value DNI -> 0.47uF; footprint Capacitor_SMD:C_0603_1608Metric -> Capacitor_SMD:C_0402_1005Metric
- C9: value 22uF -> 6.8uF; footprint Capacitor_SMD:C_0805_2012Metric -> Capacitor_SMD:C_1210_3225Metric
- D3: value PESD5V2S2UT,215 -> PESD15VL2BT,215
- L2: footprint Eros Tracker:DFE2HCAH1R0MJ0L -> Eros Tracker:1277ASH100MP2
- R11: value 100k -> 10k 1%
- R17: value 835R -> 6K65; footprint Resistor_SMD:R_0805_2012Metric -> Resistor_SMD:R_0402_1005Metric
- U3: value MCP73834-FCI/MF -> BQ24196RGER; footprint Eros Tracker:MCP73834-FCI-MF -> Eros Tracker:QFN50P400X400X100-25N-D
- moved G6 31.8 mm to (177.7, 126.9)
- moved TP8 29.4 mm to (183.2, 103.1)
- moved TP2 27.1 mm to (161.2, 108.7)
- moved L1 26.9 mm to (158.4, 110.0)
- moved C2 26.9 mm to (155.0, 107.2)
- moved U2 26.9 mm to (154.9, 110.0)
- moved C3 26.9 mm to (158.5, 107.2)
- moved R14 26.9 mm to (154.9, 111.9)
- moved R13 26.9 mm to (158.4, 111.9)
- moved R10 25.9 mm to (181.2, 94.0), turned to -90 degrees
- moved C10 22.7 mm to (150.8, 105.4), turned to 0 degrees
- moved D2 20.8 mm to (174.9, 120.0)
- moved C8 18.9 mm to (153.5, 104.9), turned to 180 degrees
- moved R11 17.4 mm to (170.2, 114.6), turned to 0 degrees
- moved C9 17.4 mm to (156.8, 102.8), turned to 0 degrees
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Connections:
- net /Eros Tracker Microcontroller/~{BUTTON_INPUT} renamed /Eros Tracker Microcontroller/BUTTON_INPUT
- C10 pad 1: /Eros Tracker Connectors/VBUS_OUT -> +4V5
- C2 pad 1: /Eros Tracker Power & Battery/VIN -> +4V5
- C8 pad 1: /Eros Tracker Connectors/VBUS_OUT -> Net-(U3-BTST)
- C8 pad 2: Net-(U5-FB) -> Net-(U3-SW)
- C9 pad 1: /Eros Tracker Connectors/VBUS_OUT -> Net-(U3-PMID)
- D1 pad 6: /Eros Tracker Microcontroller/~{BAT_STAT_CHARGING} -> /Eros Tracker Microcontroller/~{POWER GOOD}
- D2 pad 1: /Eros Tracker Power & Battery/VIN -> /Eros Tracker Connectors/VBUS_OUT
- D2 pad 2: /Eros Tracker Connectors/VBUS -> Net-(D2-A)
- FL1 pad 11: /Eros Tracker Connectors/VBUS_OUT -> unconnected-(FL1-ID-Pad4)
- FL1 pad 4: /Eros Tracker Connectors/VBUS_OUT -> unconnected-(FL1-ID-Pad4)
- J1 pad A5: Net-(J1-CC1) -> /Eros Tracker Connectors/USB_CC1
- J1 pad B5: Net-(J1-CC2) -> /Eros Tracker Connectors/USB_CC2
- L2 pad 1: /Eros Tracker Connectors/VBUS -> Net-(U3-SW)
- L2 pad 2: Net-(U5-SW) -> +4V5
- Q1 pad 2: /Eros Tracker Microcontroller/~{BAT_STAT_CHRG_DONE} -> /Eros Tracker Microcontroller/BAT_CHRG_DONE
- Q4 pad 1: /Eros Tracker Connectors/VBUS -> Net-(Q1A-D1)
- Q4 pad 5: +BATT -> /Eros Tracker Connectors/VBUS
- Q4 pad 6: /Eros Tracker Power & Battery/VIN -> Net-(D2-A)
- R10 pad 2: /Eros Tracker Microcontroller/~{BAT_STAT_CHRG_DONE} -> /Eros Tracker Microcontroller/~{POWER GOOD}
- R15 pad 1: /Eros Tracker Connectors/VBUS -> GND
- R16 pad 2: GND -> /Eros Tracker Connectors/VBUS
- R17 pad 1: Net-(U3-PROG) -> Net-(U3-REGN)
- R17 pad 2: GND -> Net-(U3-TS1)
- R18 pad 1: Net-(U3-THERM) -> Net-(U3-TS1)
- R20 pad 2: /Eros Tracker Microcontroller/~{BAT_STAT_CHARGING} -> /Eros Tracker Microcontroller/CHRG_INT
- R21 pad 1: /Eros Tracker Connectors/VBUS_OUT -> +3V3
- R21 pad 2: Net-(U5-FB) -> /Eros Tracker Microcontroller/USB_PD_INT
- TP1 pad 1: /Eros Tracker Power & Battery/VIN -> +4V5
- TP8 pad 1: /Eros Tracker Microcontroller/~{BAT_STAT_CHRG_DONE} -> /Eros Tracker Microcontroller/BAT_CHRG_DONE
- U1 pad 13: /Eros Tracker BNO086 IMU/~{RESET} -> /Eros Tracker Microcontroller/BAT_CHRG_DONE
- U1 pad 16: /Eros Tracker Microcontroller/~{BAT_STAT_CHRG_DONE} -> /Eros Tracker Microcontroller/CHRG_INT
- U1 pad 18: /Eros Tracker Microcontroller/~{BAT_STAT_CHARGING} -> /Eros Tracker Microcontroller/USB_PD_INT
- U2 pad 3: /Eros Tracker Power & Battery/VIN -> +4V5
- U2 pad 4: /Eros Tracker Power & Battery/VIN -> +4V5
- U3 pad 10: +BATT -> GND
- U3 pad 11: GND -> Net-(U3-TS1)
- U3 pad 2: /Eros Tracker Connectors/VBUS -> GND
- U3 pad 3: /Eros Tracker Microcontroller/~{BAT_STAT_CHARGING} -> /Eros Tracker Microcontroller/~{POWER GOOD}
- U3 pad 4: /Eros Tracker Microcontroller/~{BAT_STAT_CHRG_DONE} -> unconnected-(U3-STAT-Pad4)
- U3 pad 5: GND -> /Eros Tracker BNO086 IMU/I2C_SCL
- U3 pad 6: Net-(U3-PROG) -> /Eros Tracker BNO086 IMU/I2C_SDA
- U3 pad 7: GND -> /Eros Tracker Microcontroller/CHRG_INT
- U3 pad 8: Net-(U3-THERM) -> GND
- U3 pad 9: +BATT -> GND
Routing:
- net /Eros Tracker Microcontroller/~{BAT_STAT_CHRG_DONE}: track 42.1 -> 0.00 mm, vias 2 -> 0
- net /Eros Tracker Microcontroller/~{BAT_STAT_CHARGING}: track 35.0 -> 0.00 mm, vias 2 -> 0
- net /Eros Tracker Power & Battery/VIN: track 34.7 -> 0.00 mm, vias 2 -> 0
- net /Eros Tracker BNO086 IMU/I2C_SDA: track 7.66 -> 38.6 mm, vias 0 -> 2
- net /Eros Tracker Microcontroller/BAT_CHRG_DONE: track 0.00 -> 30.1 mm, vias 0 -> 2
- net +BATT: track 83.0 -> 53.4 mm
- net /Eros Tracker Microcontroller/~{POWER GOOD}: track 0.00 -> 29.1 mm, vias 0 -> 2
- net /Eros Tracker BNO086 IMU/I2C_SCL: track 7.40 -> 35.8 mm, vias 2 -> 5
- net /Eros Tracker Connectors/VBUS_OUT: track 30.7 -> 5.51 mm, vias 2 -> 1
- net +4V5: track 0.00 -> 17.9 mm, vias 0 -> 2
- net Net-(Q1A-D1): track 40.6 -> 22.9 mm, vias 3 -> 2
- net /Eros Tracker Microcontroller/USB_PD_INT: track 0.00 -> 17.1 mm, vias 0 -> 3
- net /Eros Tracker Microcontroller/ADC_BATT_V: track 21.0 -> 5.28 mm
- net Net-(U3-REGN): track 0.00 -> 15.3 mm, vias 0 -> 2
- net /Eros Tracker BNO086 IMU/INT: track 24.0 -> 10.5 mm, vias 0 -> 2
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- added copper zone on F.Cu, net +4V5
- added copper zone on F.Cu, net +BATT
- added copper zone on F.Cu, net Net-(U3-PMID)
- added copper zone on F.Cu, net Net-(U3-SW)
- removed copper zone on F.Cu, net /Eros Tracker Connectors/VBUS_OUT
- removed copper zone on F.Cu, net Net-(U5-SW)
Other:
- board text added: "Somatic Eros Rev. E"
- board text removed: "Somatic Eros Rev. D"
