File: Eros Tracker.kicad_sch (KiCad schematic)
At the start: 0 parts

Commit message: Rev D realease
Parts:
- added G1: ~, Eros Tracker:SomaticLogo, symbol Eros Tracker:LOGO_SOMATIC
- added G2: ~, Eros Tracker:SomaticBananaLogo, symbol Eros Tracker:LOGO_BANANA
- added G3: ~, Eros Tracker:CE-Logo_7.0x5.0mm_SilkScreen, symbol Eros Tracker:LOGO_CE
- added G4: ~, Eros Tracker:FCC-Logo_6.2x5.0mm_SilkScreen, symbol Eros Tracker:LOGO_FCC
- added G5: ~, Symbol:WEEE-Logo_4.2x6mm_SilkScreen, symbol Eros Tracker:LOGO_WEEE
- added G6: ~, Symbol:OSHW-Logo2_7.3x6mm_SilkScreen, symbol Eros Tracker:LOGO_OSHW
Changed lines of the file:
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@@
 (kicad_sch (version 20230121) (generator eeschema)
   (paper "A4")
-  (junction (at 118.11 100.33) (diameter 0) (color 0 0 0 0)
-  )
   (wire (pts (xy 49.53 91.44) (xy 49.53 129.54))
     (stroke (width 0) (type default))
@@
     (stroke (width 0) (type default))
   )
-  (wire (pts (xy 118.11 114.3) (xy 118.11 100.33))
-    (stroke (width 0) (type default))
-  )
-  (wire (pts (xy 118.11 71.12) (xy 118.11 100.33))
+  (wire (pts (xy 118.11 71.12) (xy 118.11 114.3))
     (stroke (width 0) (type default))
   )
@@
     (stroke (width 0) (type default))
   )
-  (wire (pts (xy 118.11 100.33) (xy 137.16 100.33))
-    (stroke (width 0) (type default))
-  )
   (wire (pts (xy 55.88 88.9) (xy 43.18 88.9))
     (stroke (width 0) (type default))
@@
   (wire (pts (xy 182.88 92.71) (xy 205.74 92.71))
     (stroke (width 0) (type default))
+  )
+  (symbol (lib_id "Eros Tracker:LOGO_SOMATIC") (at 238.76 146.05 0) (unit 1)
+    (in_bom no) (on_board yes) (dnp no) (fields_autoplaced)
+    (property "Reference" "G1" (at 238.76 143.51 0)
+      (effects (font (size 1.27 1.27)))
+    )
+    (property "Value" "~" (at 238.76 146.05 0)
+      (effects (font (size 1.27 1.27)))
+    )
+    (property "Footprint" "Eros Tracker:SomaticLogo" (at 238.76 146.05 0)
+      (effects (font (size 1.27 1.27)) hide)
+    )
+    (property "Datasheet" "" (at 238.76 146.05 0)
+      (effects (font (size 1.27 1.27)) hide)
+    )
+    (instances
+      (project "Eros Tracker"
+        (path "/e762b1f0-85b9-427f-b9a8-4b9d5ef7d00a"
+          (reference "G1") (unit 1)
+        )
+      )
+    )
   )
   (symbol (lib_id "power:GND") (at 57.15 152.4 270) (unit 1)
@@
     )
   )
+  (symbol (lib_id "Eros Tracker:LOGO_BANANA") (at 238.76 158.75 0) (unit 1)
+    (in_bom no) (on_board yes) (dnp no) (fields_autoplaced)
+    (property "Reference" "G2" (at 238.76 156.21 0)
+      (effects (font (size 1.27 1.27)))
+    )
+    (property "Value" "~" (at 238.76 158.75 0)
+      (effects (font (size 1.27 1.27)))
+    )
+    (property "Footprint" "Eros Tracker:SomaticBananaLogo" (at 238.76 158.75 0)
+      (effects (font (size 1.27 1.27)) hide)
+    )
+    (property "Datasheet" "" (at 238.76 158.75 0)
+      (effects (font (size 1.27 1.27)) hide)
+    )
+    (instances
+      (project "Eros Tracker"
+        (path "/e762b1f0-85b9-427f-b9a8-4b9d5ef7d00a"
+          (reference "G2") (unit 1)
+        )
+      )
+    )
+  )
   (symbol (lib_id "Eros Tracker-eagle-import:FRAME_A_L") (at 194.31 209.55 0) (unit 2)
     (in_bom yes) (on_board yes) (dnp no)
@@
         )
       )
+    )
+  )
+  (symbol (lib_id "Eros Tracker:LOGO_OSHW") (at 238.76 163.83 0) (unit 1)
+    (in_bom no) (on_board yes) (dnp no) (fields_autoplaced)
+    (property "Reference" "G6" (at 238.76 161.29 0)
+      (effects (font (size 1.27 1.27)))
+    )
+    (property "Value" "~" (at 238.76 163.83 0)
+      (effects (font (size 1.27 1.27)))
+    )
+    (property "Footprint" "Symbol:OSHW-Logo2_7.3x6mm_SilkScreen" (at 238.76 163.83 0)
+      (effects (font (size 1.27 1.27)) hide)
+    )
+    (property "Datasheet" "" (at 238.76 163.83 0)
+      (effects (font (size 1.27 1.27)) hide)
+    )
+    (instances
+      (project "Eros Tracker"
+        (path "/e762b1f0-85b9-427f-b9a8-4b9d5ef7d00a"
+          (reference "G6") (unit 1)
+        )
+      )
+    )
+  )
+  (symbol (lib_id "Eros Tracker:LOGO_FCC") (at 238.76 152.4 0) (unit 1)
+    (in_bom no) (on_board yes) (dnp no) (fields_autoplaced)
+    (property "Reference" "G4" (at 238.76 149.86 0)
+      (effects (font (size 1.27 1.27)))
+    )
+    (property "Value" "~" (at 238.76 152.4 0)
+      (effects (font (size 1.27 1.27)))
+    )
+    (property "Footprint" "Eros Tracker:FCC-Logo_6.2x5.0mm_SilkScreen" (at 238.76 152.4 0)
+      (effects (font (size 1.27 1.27)) hide)
+    )
+    (property "Datasheet" "" (at 238.76 152.4 0)
+      (effects (font (size 1.27 1.27)) hide)
+    )
+    (instances
+      (project "Eros Tracker"
+        (path "/e762b1f0-85b9-427f-b9a8-4b9d5ef7d00a"
+          (reference "G4") (unit 1)
+        )
+      )
+    )
+  )
+  (symbol (lib_id "Eros Tracker:LOGO_WEEE") (at 251.46 152.4 0) (unit 1)
+    (in_bom no) (on_board yes) (dnp no) (fields_autoplaced)
+    (property "Reference" "G5" (at 251.46 149.86 0)
+      (effects (font (size 1.27 1.27)))
+    )
+    (property "Value" "~" (at 251.46 152.4 0)
+      (effects (font (size 1.27 1.27)))
+    )
+    (property "Footprint" "Symbol:WEEE-Logo_4.2x6mm_SilkScreen" (at 251.46 152.4 0)
+      (effects (font (size 1.27 1.27)) hide)
+    )
+    (property "Datasheet" "" (at 251.46 152.4 0)
+      (effects (font (size 1.27 1.27)) hide)
+    )
+    (instances
+      (project "Eros Tracker"
+        (path "/e762b1f0-85b9-427f-b9a8-4b9d5ef7d00a"
+          (reference "G5") (unit 1)
+        )
+      )
+    )
+  )
+  (symbol (lib_id "Eros Tracker:LOGO_CE") (at 227.33 152.4 0) (unit 1)
+    (in_bom no) (on_board yes) (dnp no)
+    (property "Reference" "G3" (at 227.33 149.86 0)
+      (effects (font (size 1.27 1.27)))
+    )
+    (property "Value" "~" (at 227.33 152.4 0)
+      (effects (font (size 1.27 1.27)))
+    )
+    (property "Footprint" "Eros Tracker:CE-Logo_7.0x5.0mm_SilkScreen" (at 227.33 152.4 0)
+      (effects (font (size 1.27 1.27)) hide)
+    )
+    (property "Datasheet" "" (at 227.33 152.4 0)
+      (effects (font (size 1.27 1.27)) hide)
+    )
+    (instances
+      (project "Eros Tracker"
+        (path "/e762b1f0-85b9-427f-b9a8-4b9d5ef7d00a"
+          (reference "G3") (unit 1)
+        )
+      )

Commit message: Rev E release
Other:
- sheet Eros Tracker Connectors ports: added USB_CC1, USB_CC2; removed none
- sheet Eros Tracker Microcontroller ports: added BAT_CHRG_DONE, CHRG_INT, USB_CC1, USB_CC2, VBUS, ~{POWER GOOD}; removed IMU_RESET, ~{BAT_STAT_CHARGING}, ~{BAT_STAT_CHRG_DONE}
- sheet Eros Tracker Power & Battery ports: added BAT_CHRG_DONE, CHRG_INT, I2C_SCL, I2C_SDA, ~{POWER GOOD}; removed ~{BAT_STAT_CHARGING}, ~{BAT_STAT_CHRG_DONE}
